Commit message: done mo phong

File: src/ur5_description/urdf/ur5.xacro (robot description, xacro)
@@ -11,5 +11,5 @@
     <inertial>
       <mass value="${mass}" />
-      <inertia ixx="0.1" ixy="0.0" ixz="0.0" iyy="0.1" iyz="0.0" izz="0.1" />
+      <inertia ixx="1.0" ixy="0.0" ixz="0.0" iyy="1.0" iyz="0.0" izz="1.0" />
     </inertial>
   </xacro:macro>
@@ -18,5 +18,5 @@
     <parent link="world" />
     <child link = "base_link" />
-    <origin xyz="0.0 0.0 0.0" rpy="0.0 0.0 0.0" />
+    <origin xyz="0.0 0.0 1.0" rpy="0.0 0.0 0.0" />
   </joint>
   <link name="base_link">
@@ -31,4 +31,5 @@
   </link>
   <joint name="shoulder_pan_joint" type="revolute">
+    <dynamics damping="1000.0" friction="1000.0"/>
     <parent link="base_link" />
     <child link = "shoulder_link" />
@@ -47,4 +48,5 @@
   </link>
   <joint name="shoulder_lift_joint" type="revolute">
+    <dynamics damping="1000.0" friction="1000.0"/>
     <parent link="shoulder_link" />
     <child link = "upper_arm_link" />
@@ -63,4 +65,5 @@
   </link>
   <joint name="elbow_joint" type="revolute">
+    <dynamics damping="1000.0" friction="1000.0"/>
     <parent link="upper_arm_link" />
     <child link = "forearm_link" />
@@ -79,4 +82,5 @@
   </link>
   <joint name="wrist_1_joint" type="revolute">
+    <dynamics damping="10.0" friction="1.0"/>
     <parent link="forearm_link" />
     <child link = "wrist_1_link" />
@@ -95,4 +99,5 @@
   </link>
   <joint name="wrist_2_joint" type="revolute">
+    <dynamics damping="10.0" friction="1.0"/>
     <parent link="wrist_1_link" />
     <child link = "wrist_2_link" />
@@ -111,4 +116,5 @@
   </link>
   <joint name="wrist_3_joint" type="revolute">
+    <dynamics damping="10.0" friction="1.0"/>
     <parent link="wrist_2_link" />
     <child link = "wrist_3_link" />
@@ -126,17 +132,59 @@
     <xacro:default_inertial mass="${wrist_3_mass}"/>
   </link>
-  <joint name="gripper_joint" type="fixed">
+  <joint name="rg2_joint" type="fixed">
     <parent link="wrist_3_link" />
-    <child link = "gripper_link" />
-    <origin xyz="0.0 0.08 0.0" rpy="1.57 0 0" /> </joint>
-  <link name="gripper_link">
+    <child link = "rg2_base_link" />
+    <origin xyz="0.0 0.08 0.0" rpy="1.5708 0 -1.5708" />
+  </joint>
+  <link name="rg2_base_link">
     <visual>
-      <geometry><box size="0.05 0.12 0.05"/></geometry>
-      <material name="Black"><color rgba="0.1 0.1 0.1 1.0"/></material>
+      <geometry>
+        <mesh filename="package://ur5_description/meshes/rg2/rg2_base.dae" scale="1.0 1.0 1.0"/>
+      </geometry>
+      <material name="Grey"><color rgba="0.5 0.5 0.5 1"/></material>
     </visual>
     <collision>
-      <geometry><box size="0.05 0.12 0.05"/></geometry>
+      <geometry>
+         <mesh filename="package://ur5_description/meshes/rg2/rg2_base.dae" scale="1.0 1.0 1.0"/>
+      </geometry>
     </collision>
-    <xacro:default_inertial mass="0.5"/>
+    <xacro:default_inertial mass="0.2"/>
+  </link>
+  <joint name="rg2_finger1_joint" type="fixed">
+    <parent link="rg2_base_link" />
+    <child link = "rg2_finger1_link" />
+    <origin xyz="0.017 0.05 0.0" rpy="0 0 -0.5" />
+  </joint>
+  <link name="rg2_finger1_link">
+    <visual>
+      <geometry>
+        <mesh filename="package://ur5_description/meshes/rg2/rg2_finger.dae" scale="1.0 1.0 1.0"/>
+      </geometry>
+      <material name="DarkGrey"><color rgba="0.2 0.2 0.2 1"/></material>
+    </visual>
+    <collision>
+      <geometry>
+        <mesh filename="package://ur5_description/meshes/rg2/rg2_finger.dae" scale="1.0 1.0 1.0"/>
+      </geometry>
+    </collision>
+    <xacro:default_inertial mass="0.05"/>
+  </link>
+  <joint name="rg2_finger2_joint" type="fixed">
+    <parent link="rg2_base_link" />
+    <child link = "rg2_finger2_link" />
+    <origin xyz="-0.017 0.05 0.0" rpy="0 0 3.64" /> </joint>
+  <link name="rg2_finger2_link">
+    <visual>
+      <geometry>
+        <mesh filename="package://ur5_description/meshes/rg2/rg2_finger.dae" scale="1.0 1.0 1.0"/>
+      </geometry>
+      <material name="DarkGrey"/>
+    </visual>
+    <collision>
+      <geometry>
+        <mesh filename="package://ur5_description/meshes/rg2/rg2_finger.dae" scale="1.0 1.0 1.0"/>
+      </geometry>
+    </collision>
+    <xacro:default_inertial mass="0.05"/>
   </link>
   <gazebo>
